File: EHI/Power_Stage.kicad_sch (KiCad schematic)
At the start: 31 parts

Commit message: new
Parts:
- removed Q?: IRFZ44N, TO-220, symbol EESTN5:IRFZ44N
- removed Q? (x2): 2N7002, symbol EESTN5:2N7002
- removed R? (x8): R, symbol EESTN5:R
Connections:
- net PW_H is gone; now on net GND: D?.1 (A), D?.1 (A), Q?.3 (S), Q?.3 (S)
Other:
- moved on the sheet: D?, J?, Q?, R?
