File: EHI/Protection.kicad_sch (KiCad schematic)
At the start: 21 parts

Commit message: actualizacion del proteyecto Olimpiadas
Parts:
- removed R? (x6): R, symbol EESTN5:R
- removed U? (x2): LM324, symbol MacroLib:LM324
- added 100uf?: C, symbol EESTN5:C
- added 1N? (x2), S5AC?: DIODE, symbol EESTN5:DIODE
- added ENTRADA-12V?, SALIDA-12V?: TB_1X2, symbol EESTN5:TB_1X2
- added LED?: LED, symbol EESTN5:LED
- added Q?: BC558, TO92260P520H933-3, symbol BC558:BC558
- added R?: 100k, symbol EESTN5:R
- added R?: 510, symbol EESTN5:R
- added U?: FUSIBLE, symbol EESTN5:FUSIBLE
- R1, R2, R4, R5: renamed from R?; value R -> 1k5
- R3, R6: renamed from R?; value R -> 10k
Connections:
- net GND: now also 100uf?.2, ENTRADA-12V?.1, R?.1, R?.2, S5AC?.1 (A), SALIDA-12V?.2
- net RT1: now also U?.13 (-)
- net RT2: no longer U?.13 (-)
- new net: ENTRADA-12V?.2, LED?.1 (A), U?.1
- new net: 1N?.1 (A), 1N?.1 (A), S5AC?.2 (K), U?.2
- new net: 100uf?.1, 1N?.2 (K), SALIDA-12V?.1
- new net: 1N?.2 (K), Q?.2, R?.1
- new net: Q?.1, R?.2
- new net: LED?.2 (K), Q?.3
Other:
- note added: "ENTRADA 12V"
- note added: "FALLA FUSIBLE"
- note added: "FILTRO"
- note added: "PROTECCIONES"
- note added: "SALIDA 12V"
- moved on the sheet: R?, U?

Commit message: new
Parts:
- removed 100uf?: C, symbol EESTN5:C
- removed 1N?: DIODE, symbol EESTN5:DIODE
- removed SALIDA-12V?: TB_1X2, symbol EESTN5:TB_1X2
- removed U?: FUSIBLE, symbol EESTN5:FUSIBLE
Connections:
- net NTC2: now also R3.1, U?.8; no longer R6.1, U?.14
- net +12V: now reaches 1N?.1 (A), S5AC?.2 (K), U?.2
- new net NTC1: R6.1, U?.14
Other:
- note removed: "FILTRO"
- note removed: "SALIDA 12V"
- moved on the sheet: 1N?, ENTRADA-12V?, LED?, Q?, R1, R2, R3, R4, R5, R6, R?, S5AC?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
